File: hardware/PCB/bitchess.brd (EAGLE design)
At the start: 85 x 52.2 mm, 7 parts, among them CON3 A2600

Commit message: randomised board. gcode.
Routing:
- net D6: track 79.6 -> 75.1 mm
- net D7: track 77.3 -> 78.7 mm
Other:
- board text added: "/Users/boo/Desktop/front.bmp"

Commit message: no idea if this is OK, but committing to tidy up
Routing:
- net D7: track 78.7 -> 84.0 mm
- net +3V3: track 112.0 -> 113.0 mm
- net A10: track 85.6 -> 86.5 mm
- net A9: track 87.6 -> 88.4 mm
- net A12: track 82.1 -> 82.8 mm
- net A8: track 95.4 -> 96.1 mm
- net A11: track 84.3 -> 85.0 mm
